File: The Button/The Button.kicad_pcb (KiCad board)
At the start: 2 copper layers, 54 x 74 mm, 28 parts, among them J1 Gnd, J2 2169890001, J3 Extra Pins, J4 Buttons, J5 Conn_01x05_Pin, SW8 SW_SPST BOOT, U1 LD1117S33TR_SOT223, U2 STM32C071KBTx, U5 USBLC6-2SC6

Commit message: Move character conversion to separate file
Parts:
- moved D3 1.14 mm to (176.5, 96.5)
Connections:
- U2 pad 10: GND -> unconnected-(U2-PA3-Pad10)
Routing:
- net GND: track 6.08 -> 1.99 mm, vias 29 -> 31
- net Net-(D3-K): track 2.08 -> 3.79 mm, vias 0 -> 2
- net USR_LED_2: track 30.7 -> 31.5 mm
Other:
- board text added: "GND PA2 PA1 PA0"
- board text added: "Key Hi Lo Gnd"
- board text added: "The Button v2 by Maebe.me"
